File: enchantiS3T-board/enchantiS3T.kicad_pcb (KiCad board)
At the start: 4 copper layers, 55.9 x 31.8 mm, 64 parts, among them J1 USB_C_Receptacle_USB2.0, J2 Conn_01x03_MountingPin, J3 Progamming Header, J4 BC075-03-A-L-A_REVC2, J5 BC075-03-A-L-A_REVC2, SW1 B3U-1000P, SW2 B3U-1000P, U1 USBLC6-2P6, U10 BQ25185DLHR, U11 PTCAN3413DRBR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

Commit message: finsished routing for revision 4 of enchantiS3, finished routing for  enchantiS3 Touch
Parts:
- removed J4, J5: BC075-03-A-L-A_REVC2, BC075-footprint:GCT_BC075-03-A-L-A_REVC2
- added FP1: JST-SH-1x04 1.0mm, Connector_JST:JST_SH_BM06B-SRSS-TB_1x06-1MP_P1.00mm_Vertical, F.Cu at (120.4, 73.8)
- moved U2 36.2 mm to (147.4, 50.3), turned to -90 degrees
- moved C18 36.1 mm to (145.4, 50.0)
- moved R4 19.4 mm to (143.7, 57.4), turned to 0 degrees
- moved R9 17.9 mm to (141.8, 57.4), turned to 180 degrees
- moved U11 2.41 mm to (116.9, 67.8)
- moved C4 1.87 mm to (106.3, 67.0), turned to 90 degrees
- moved C26 1.35 mm to (120.7, 69.2)
- moved C27 1.35 mm to (119.7, 69.2)
Connections:
- U3 pad 3: SYS -> /LDO_EN
- U3 pad 4: /LDO_EN -> SYS
- U9 pad 28: /ORANGELED -> /LED2
- U9 pad 29: /BLUELED -> /LED1
- U9 pad 31: /SCL2 -> unconnected-(U9-SPIIO6/GPIO35/FSPID/SUBSPID-Pad31)
- U9 pad 32: /SDA2 -> unconnected-(U9-SPIIO7/GPIO36/FSPICLK/SUBSPICLK-Pad32)
- U9 pad 5: /IO1 -> /SCL2
- U9 pad 6: /IO2 -> /SDA2
Routing:
- net /BLUELED: track 46.1 -> 0.00 mm, vias 4 -> 0
- net /ORANGELED: track 45.9 -> 0.00 mm, vias 4 -> 0
- net /LED2: track 0.00 -> 16.6 mm, vias 0 -> 2
- net /LED1: track 0.00 -> 14.1 mm
- net /BTN: track 25.6 -> 14.8 mm
- net 3V3_AUX: track 127.0 -> 118.7 mm
- net GND: track 92.2 -> 86.5 mm, vias 31 -> 32
- net /SDA2: track 16.5 -> 10.9 mm, vias 0 -> 2
- net /SCL2: track 15.8 -> 10.6 mm, vias 0 -> 2
- net /STAT2: track 22.5 -> 27.4 mm, vias 2 -> 4
- net SYS: track 27.5 -> 30.9 mm
- net /CANFD_TX: track 11.6 -> 13.3 mm
- net /CANFD_RX: track 9.21 -> 10.8 mm
- net /CAN_MODE: track 19.2 -> 20.0 mm
- net /STAT1: track 19.1 -> 19.7 mm
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Other:
- board text removed: "FP1"
- board text removed: "FP2"
