File: enchantiS3T-board/enchantiS3T.kicad_sch (KiCad schematic)
At the start: 69 parts, among them J1 USB_C_Receptacle_USB2.0, J2 Conn_01x03_MountingPin, J3 Progamming Header, J4 BC075-03-A-L-A_REVC2, J5 BC075-03-A-L-A_REVC2, SW1 B3U-1000P, SW2 B3U-1000P, U1 USBLC6-2P6, U10 BQ25185DLHR, U11 PTCAN3413DRBR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

Commit message: finsished routing for revision 4 of enchantiS3, finished routing for  enchantiS3 Touch
Parts:
- removed J4, J5: BC075-03-A-L-A_REVC2, BC075-footprint:GCT_BC075-03-A-L-A_REVC2, symbol BC075-03-A-L-A_REVC2:BC075-03-A-L-A_REVC2
- added FP1: JST-SH-1x04 1.0mm, Connector_JST:JST_SH_BM06B-SRSS-TB_1x06-1MP_P1.00mm_Vertical, symbol Connector_Generic_MountingPin:Conn_01x06_MountingPin
Connections:
- net IO1 is gone; now on net SCL2: U9.5 (GPIO1/TOUCH1/ADC1_CH0)
- net IO2 is gone; now on net SDA2: U9.6 (GPIO2/TOUCH2/ADC1_CH1)
- net 3V3_AUX: now also FP1.1 (Pin_1)
- net BTN: now also FP1.2 (Pin_2)
- net GND: now also FP1.MP (MountPin)
- net LDO_EN: now also U3.3 (EN); no longer U3.4 (IN)
- net SCL2: no longer U9.31 (SPIIO6/GPIO35/FSPID/SUBSPID)
- net SDA2: no longer U9.32 (SPIIO7/GPIO36/FSPICLK/SUBSPICLK)
- net STAT1: now also FP1.6 (Pin_6)
- net STAT2: now also FP1.5 (Pin_5)
- net SYS: now also U3.4 (IN); no longer U3.3 (EN)
- net BLUELED renamed LED1
- net LED1: now also FP1.3 (Pin_3)
- net ORANGELED renamed LED2
- net LED2: now also FP1.4 (Pin_4)
Other:
- note added: "Connect to Frontplate"
- note removed: "BLUE LED == Connected to Wifi"
- note removed: "ORANGE LED == Setting up/Fail State"
- moved on the sheet: C4
