File: enchanti-Module/enchanti-module.kicad_pcb (KiCad board)
At the start: 4 copper layers, 46 x 46 mm, 82 parts, among them J1 878-22-004-10-011101, J2 Programming Header, J3 USB_C_Receptacle_USB2.0, U1 Sona-IF573, U10 ICM-42670-P, U12 MMC5633NJL, U13 B3U-1000P, U2 STM32H7R3V8T6, U3 NCP167AMX180TBG, U4 B3U-1000P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

Commit message: removed unused nets, simplified connector
Parts:
- removed R15, R16: 1k, Resistor_SMD:R_0402_1005Metric
- removed STATLED1: GENERAL STATUS, LED_SMD:LED_0402_1005Metric
- removed STATLED2: WIFISTATUS, LED_SMD:LED_0402_1005Metric
- added R27: 10k, Resistor_SMD:R_0402_1005Metric, B.Cu at (87.7, 70.3)
- added U7: LM66200DRLR, ENCHANTI_regulators:SOT-5X3_DRL_TEX, B.Cu at (86.5, 72.3)
- J1: value 878-22-004-10-011101 -> Enchanti-Module-Receptacle; footprint ENCHANTI_connectors:CONN_878-22-004-10-011101_MIM -> ENCHANTI_connectors:Enchanti-Module-Receptacle
- U6: footprint ENCHANTI_regulators:NCV8187AMT330TAG_ONS -> ENCHANTI_regulators:NCV8187AMT330TAG_ONS-L
- moved D1 24.8 mm to (91.4, 72.1), turned to 90 degrees
- moved U13 20.4 mm to (93.3, 76.5), turned to 0 degrees
- moved R14 19.0 mm to (94.4, 78.5)
- moved R8 17.7 mm to (92.0, 78.5), turned to 0 degrees
- moved J1 3.70 mm to (90.4, 76.2)
- moved U10 1.63 mm to (75.3, 83.8)
- moved C37 0.91 mm to (72.7, 83.3), turned to 180 degrees
- moved C29 0.38 mm to (96.0, 81.9)
- moved R19 0.36 mm to (86.9, 88.6)
- moved R20 0.35 mm to (86.8, 86.0)
Connections:
- J1 pad 1: SYS -> +5V
- J1 pad 2: /CAN_H -> /CAN_L
- J1 pad 3: /CAN_L -> /CAN_H
- U2 pad 75: /INT_LEDB -> unconnected-(U2A-PM2-Pad75)
- U2 pad 76: /INT_LEDO -> unconnected-(U2A-PM3-Pad76)
Routing:
- net VUSB: track 16.1 -> 44.5 mm, vias 2 -> 4
- net /CAN_L: track 3.09 -> 27.5 mm
- net /CAN_H: track 2.95 -> 26.9 mm
- net GND: track 52.9 -> 71.2 mm, vias 19 -> 29
- net +1V8: track 201.9 -> 215.8 mm, vias 19 -> 20
- net +5V: track 0.00 -> 10.2 mm
- net /BT_REG_ON: track 10.0 -> 18.2 mm
- net Net-(R14-Pad2): track 0.00 -> 4.24 mm
- net SYS: track 20.9 -> 23.4 mm, vias 1 -> 3
- net /I3C_SCL: track 22.0 -> 19.8 mm
- net /SDMMC_D3: track 11.5 -> 13.5 mm
- net /BOOT: track 0.00 -> 1.97 mm
- net /INT_LEDB: track 1.72 -> 0.00 mm, vias 1 -> 0
- net /INT_LEDO: track 1.68 -> 0.00 mm, vias 1 -> 0
- net /SDMMC_D2: track 11.3 -> 12.8 mm
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