File: enchanti-Module/enchanti-module.kicad_sch (KiCad schematic)
At the start: 97 parts, among them J1 USB_C_Receptacle_USB2.0, J2 Programming Header, J3 Programming Header, SW2 KSC441G DCT 70SH LFS, U1 BQ25185DLHR, U10 ICM-42670-P, U11 IRIS-W106-30B, U12 MMC5633NJL, U2 STM32H7R3V8T6, U3 NCP167AMX180TBG, U4 B3U-1000P, U5 NCP167AMX330TBG, U6 USBLC6-2P6, U7 MAX17262REWL+T, U8 S76HS512TC0BHB010, U9 TCAN3413DRBR

Commit message: added usb connector, added leds
Parts:
- removed C31: 0.1uF, Capacitor_SMD:C_0402_1005Metric, symbol Device:C
- removed FP1: JST-SH-1x04 1.0mm, Connector_JST:JST_SH_BM06B-SRSS-TB_1x06-1MP_P1.00mm_Vertical, symbol Connector_Generic_MountingPin:Conn_01x06_MountingPin
- removed J1: USB_C_Receptacle_USB2.0, Connector_USB:USB_C_Receptacle_GCT_USB4105-xx-A_16P_TopMnt_Horizontal, symbol Connector:USB_C_Receptacle_USB2.0
- removed SW2: KSC441G DCT 70SH LFS, ENCHANTI_switches:KSC-DCT_6P2X6P2_CNK, symbol ENCHANTI_switches:KSC441G_DCT_70SH_LFS
- removed SYS5, SYS6: SYS, symbol power-symbols:VSYS
- removed TP1: CHRG TP, TestPoint:TestPoint_Pad_D1.0mm, symbol Connector:TestPoint
- added D2, D3: RGB-LED, ENCHANTI_leds:LED_APFA3010LSEEZGKQBKC, symbol ENCHANTI_leds:APFA3010LSEEZGKQBKC
- added J5: CONN_MEZANNINE, ENCHANTI_connectors:CON_536250674_MOL, symbol ENCHANTI_connectors:Module_Connector
- added R31: 1k, Resistor_SMD:R_0402_1005Metric, symbol Device:R_US
- added U13: B3U-1000P, ENCHANTI_switches:B3U-1000P, symbol ENCHANTI_switches:B3U-1000P
- added USB1: GSB1CA11101DSHR, ENCHANTI_connectors:AMPHENOL_GSB1CA11101DSHR, symbol ENCHANTI_connectors:GSB1CA11101DSHR
- R10, R8: value 10k -> 1k; Mfg Part # ERJ-2RKF1002X -> ERJ-2RKF1001X
- U11: value IRIS-W106-30B -> IRIS-W106-00B; Mfg Part # IRIS-W106-30B -> IRIS-W106-00B
Connections:
- net CE is gone; now on net GND: U1.4 (/CE)
- net RES is gone; now on net JTAG_nRST: J3.10 (RES)
- net SWDA is gone; now on net JTAG_TMS: J3.2 (SWDIO)
- net +1V8: now also J5.39 (Pin_39), U13.2; no longer R10.1, R8.1
- net +3V3: now also R10.1, J5.9 (Pin_9)
- net +BATT: now also J5.31 (Pin_31), J5.32 (Pin_32), J5.33 (Pin_33), J5.34 (Pin_34), J5.35 (Pin_35), J5.36 (Pin_36), J5.37 (Pin_37), J5.38 (Pin_38)
- net BOOT: now also R8.1; no longer R14.1
- net BTN1: now also U2.99 (PB8), J5.15 (Pin_15); no longer U2.18 (PA2)
- net BTN2: now also U2.100 (PB9), J5.16 (Pin_16); no longer U2.19 (PA3)
- net CAN_H: now also D1.1 (K), J5.40 (Pin_40); no longer D1.2 (K)
- net CAN_L: now also D1.2 (K), J5.41 (Pin_41); no longer D1.1 (K)
- net CAN_MODE: now also U2.61 (PA10); no longer U2.74 (PM1)
- net D+: now also USB1.A6 (DP1), USB1.B6 (DP2)
- net D-: now also USB1.A7 (DN1), USB1.B7 (DN2)
- net EN_3V3REG: now also U2.74 (PM1); no longer U2.73 (PM0)
- net FSR1: now also J5.21 (Pin_21)
- net FSR2: now also J5.22 (Pin_22)
- net GND: now also R14.1, D3.3, J5.26 (Pin_26), J5.27 (Pin_27), J5.28 (Pin_28), J5.29 (Pin_29), J5.30 (Pin_30), J5.56 (Pin_56), J5.57 (Pin_57), J5.58 (Pin_58), J5.59 (Pin_59), J5.60 (Pin_60), USB1.A1 (GND), USB1.A12 (GND), USB1.B1 (GND), USB1.B12 (GND), USB1.SH (SHIELD)
- net I2C2_SCL: now also J5.43 (Pin_43)
- net I2C2_SDA: now also J5.42 (Pin_42)
- net JTDI: now also J5.54 (Pin_54); no longer J2.8 (TDI), U2.66 (PA15)
- net JTDO: now also J5.53 (Pin_53); no longer J2.6 (SWO)
- net LED1: now also U2.2 (PC13), J5.17 (Pin_17); no longer U2.21 (PA4)
- net LED2: now also U2.60 (PA9), U2.93 (PB5), J5.18 (Pin_18); no longer U2.22 (PA5)
- net NRST: now also J5.55 (Pin_55)
- net STAT1: now also D3.1, J5.19 (Pin_19)
- net STAT2: now also D3.4, J5.20 (Pin_20)
- net SWCLK: now also J5.52 (Pin_52); no longer J3.4 (SWCLK)
- net SWDIO: now also J5.51 (Pin_51)
- net USBD+: now also J5.44 (Pin_44)
- net USBD-: now also J5.45 (Pin_45)
- net VUSB: now also J5.1 (Pin_1), J5.2 (Pin_2), J5.3 (Pin_3), J5.4 (Pin_4), J5.5 (Pin_5), J5.6 (Pin_6), J5.7 (Pin_7), J5.8 (Pin_8), R31.1, USB1.A4 (VBUS), USB1.A9 (VBUS), USB1.B4 (VBUS), USB1.B9 (VBUS)
- net at R14.2: now also R8.2, U13.1
- net at U8.A4 (RESET#): no longer R8.2
- net JTAG_TDO: now reaches U11.A12 (JTAG_TDO)
- net JTAG_TDO: now also J3.6 (SWO), J5.48 (Pin_48)
- net JTAG_TMS: now reaches U11.A14 (JTAG_TMS)
- net JTAG_TMS: now also J5.46 (Pin_46)
- net JTAG_nRST: now reaches U11.B11 (JTAG_nRST)
- net JTAG_nRST: now also J5.50 (Pin_50)
- net JTAG_TDI: now reaches U11.B12 (JTAG_TDI)
- net JTAG_TDI: now also J3.8 (TDI), J5.49 (Pin_49)
- net JTAG_TCK: now reaches U11.B14 (JTAG_TCK)
- net JTAG_TCK: now also J3.4 (SWCLK), J5.47 (Pin_47)
- net at R7.2: now also USB1.A5 (CC1)
- net at R6.2: now also USB1.B5 (CC2)
- net I2S6_SDI/SPI1_MISO: now reaches U2.24 (PA6)
- net I2S6_SDI/SPI1_MISO: now also J5.13 (Pin_13)
- net I2S6_SDO/SPI1_MOSI: now reaches U2.25 (PA7)
- net I2S6_SDO/SPI1_MOSI: now also J5.14 (Pin_14)
- net ANG1: now reaches U2.26 (PB0)
- net ANG1: now also J5.23 (Pin_23)
- net ANG2: now reaches U2.27 (PB1)
- net ANG2: now also J5.24 (Pin_24)
- net ANG3: now reaches U2.28 (PB2)
- net ANG3: now also J5.25 (Pin_25)
- net INT_LED1 renamed INT_LEDB
- net INT_LED2 renamed INT_LEDO
- removed net RSTO#: R10.2, U2.89 (PM13), U8.A2 (RSTO#)
- new net: D2.2, R10.2
- new net: D3.2, R31.2
- new net I2S6_CK/SPI1_SCK: J5.12 (Pin_12), U2.22 (PA5)
- new net I2S6_MCK: J5.10 (Pin_10), U2.19 (PA3)
- new net I2S6_WS/SPI1_NSS: J5.11 (Pin_11), U2.21 (PA4)
- new net LEDB: D2.4
- new net LEDR: D2.1, D2.3
- no-connect marks 98 -> 105
Other:
- note added: "Mezannine Connector"
- note removed: "4 pin cable (pico clasp)"
- note removed: "5V 150mA buck Boost (LEDs + touch)"
- note removed: "Backplane Spring-loaded terminals"
- note removed: "Frontplate Connector Socket"
- moved on the sheet: C23, C37, J3, R15, R16, R6, R7, STATLED1, STATLED2, U12, U6

Commit message: added battery module, initial routing for power and data traces
Parts:
- removed C23: 0.1uF, Capacitor_SMD:C_0402_1005Metric, symbol Device:C
- removed C24: 0.47uF, Capacitor_SMD:C_0402_1005Metric, symbol Device:C
- removed C33: 1uF, Capacitor_SMD:C_0402_1005Metric, symbol Device:C
- removed CHARGLED1: S1, LED_SMD:LED_0402_1005Metric, symbol Device:LED
- removed D2, D3: RGB-LED, ENCHANTI_leds:LED_APFA3010LSEEZGKQBKC, symbol ENCHANTI_leds:APFA3010LSEEZGKQBKC
- removed J3: Programming Header, ENCHANTI_connectors:SAMTEC_FTSH-105-01-F-DV-P-TR, symbol ENCHANTI_connectors:Programming_Header
- removed R24: 47k, Resistor_SMD:R_0402_1005Metric, symbol Device:R_US
- removed R26, R27, R28, R29, R30: 30, Resistor_SMD:R_0402_1005Metric, symbol Device:R_US
- removed R31: 1k, Resistor_SMD:R_0402_1005Metric, symbol Device:R_US
- removed U1: BQ25185DLHR, ENCHANTI_battery-management:WSON10_DLH_TEX, symbol ENCHANTI_battery-management:BQ25185DLHR
- removed U11: IRIS-W106-00B, ENCHANTI_WiFi:IRIS-W106, symbol ENCHANTI_WiFi:IRIS-W106
- removed U5: NCP167AMX330TBG, ENCHANTI_regulators:XDFN4_1X1_711AJ_ONS, symbol ENCHANTI_regulators:NCP167AMX330TBG
- removed U6: USBLC6-2P6, Package_TO_SOT_SMD:SOT-666, symbol Power_Protection:USBLC6-2P6
- removed U7: MAX17262REWL+T, ENCHANTI_battery-management:MAX17262, symbol ENCHANTI_battery-management:MAX17262REWL+T
- removed USB1: GSB1CA11101DSHR, ENCHANTI_connectors:AMPHENOL_GSB1CA11101DSHR, symbol ENCHANTI_connectors:GSB1CA11101DSHR
- added PGLED1: PGLED1, LED_SMD:LED_0402_1005Metric, symbol Device:LED
- added PGLED2: S1, LED_SMD:LED_0402_1005Metric, symbol Device:LED
- added U1: Sona-IF573, ENCHANTI_WiFi:Sona-IF573, symbol ENCHANTI_wifi:Sona-IF573
- added U6: NCP187AMT330TAG, ENCHANTI_regulators:NCV8187AMT330TAG_ONS, symbol ENCHANTI_regulators:NCP187AMT330TAG
- added XTAL3: SIT1552AC-JE-DCC-32.768E, ENCHANTI_crystal-resonators:BGA4_SiT1532_SIT, symbol ENCHANTI_crystals-resonators:SIT1552AC-JE-DCC-32.768E
- C13: value 0.1uF -> 10uF; footprint Capacitor_SMD:C_0402_1005Metric -> Capacitor_SMD:C_0603_1608Metric; Mfg Part # CL05B104KO5NNNC -> CL10A106KO8NNNC; mpn (none) -> CL10A105KO8NNNC
- C20, C3: value 1uF -> 10uF; footprint Capacitor_SMD:C_0402_1005Metric -> Capacitor_SMD:C_0603_1608Metric; Mfg Part # CL05A105KO5NNNC -> CL10A106KO8NNNC; mpn CL05A105KO5NNNC -> CL10A105KO8NNNC
- J5: now in the parts list
- R11: value 1k -> 10k; Mfg Part # ERJ-2RKF1001X -> ERJ-2RKF1002X
- R12, R13: value 2k2 -> 30; Description Value Pkg 2.2 kOhms ±1% 0.1W, 1/10W Chip Resistor 0402 (1005 Metric) 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 -> (none); Mfg Part # ERJ-2RKF2201X -> ERJ-2RKF30R0X; mpn ERJ-2RKF2201X -> (none)
- R17: mpn ERJ-2RKF1001X -> (none)
- R2: value 13k -> 10k; Mfg Part # ERJ-2RKF1302X -> ERJ-2RKF1002X; mpn ERJ-2RKF2201X -> ERJ-2RKF1001X
- R21, R22, R23: value 47k -> 10k; Mfg Part # ERJ-2RKF4702X -> ERJ-2RKF1002X
- R3: value 0.43k -> 10k; Mfg Part # ERJ-2RKF4300X -> ERJ-2RKF1002X; mpn ERJ-2RKF2201X -> ERJ-2RKF1001X
- R4: value 10k -> 30; Mfg Part # ERJ-2RKF1002X -> ERJ-2RKF30R0X; mpn ERJ-2RKF1001X -> (none)
- R6, R7: value 5k1 -> 30; Mfg Part # ERJ-2RKF5101X -> ERJ-2RKF30R0X; mpn ERJ-2RKF5101X -> (none)
Connections:
- net CHRG+ is gone; now on net +3V3: C3.1
- net ISET is gone; now on net GND: R3.2
- net JTAG_nRST is gone; now on net I2S6_SDO/SPI1_MOSI: J5.50 (Pin_50)
- net JTDI is gone; now on net I2S6_MCK: J5.54 (Pin_54)
- net JTDO is gone; now on net I2S6_WS/SPI1_NSS: J5.53 (Pin_53)
- net PDn is gone; now on net SDMMC_D3: R17.2
- net TMR is gone; now on net SDMMC_CMD: R4.2
- net VSET is gone; now on net +1V8: R2.2
- net +1V8: now also J5.56 (Pin_56), R17.1, PGLED2.2 (A), U1.42 (VDDIO), XTAL3.3 (VDD); no longer J5.39 (Pin_39), R12.2, R13.2
- net +3V3: now also C1.1, C13.1, C5.1, J5.26 (Pin_26), R11.1, U1.4 (VBAT), U1.5 (VBAT), U1.72 (VBAT), U1.73 (VBAT), U6.5 (SNS), U6.6 (OUT); no longer J5.9 (Pin_9), R10.1, R17.1
- net ANG1: now also J5.18 (Pin_18); no longer J5.23 (Pin_23), U2.26 (PB0)
- net ANG2: now also J5.19 (Pin_19); no longer J5.24 (Pin_24)
- net ANG3: now also J5.20 (Pin_20); no longer J5.25 (Pin_25)
- net BTN1: no longer J5.15 (Pin_15)
- net BTN2: no longer J5.16 (Pin_16)
- net FSR1: now also J5.16 (Pin_16); no longer J5.21 (Pin_21)
- net FSR2: now also J5.17 (Pin_17); no longer J5.22 (Pin_22)
- net GND: now also R10.2, U1.17 (GND), U1.20 (GND), U1.23 (GND), U1.25 (JTAG_SEL), U1.26 (GND), U1.32 (GND), U1.35 (GND), U1.38 (GND), U1.41 (GND), U1.6 (GND), U1.62 (GND), U1.68 (GND), U1.71 (GND), U1.74 (GND), U1.75 (GND), U1.76 (GND), U1.77 (GND), U1.78 (GND), U1.80 (GND), U1.81 (GND), U1.82 (GND), U1.83 (GND), U1.84 (GND), U1.85 (GND), U1.87 (GND), U1.88 (GND), U1.89 (GND), U1.90 (GND), U1.91 (GND), U1.92 (GND), U1.93 (GND), U1.95 (GND), U1.96 (GND), U1.G1 (GND), U1.G10 (GND), U1.G11 (GND), U1.G12 (GND), U1.G2 (GND), U1.G3 (GND), U1.G4 (GND), U1.G5 (GND), U1.G6 (GND), U1.G7 (GND), U1.G8 (GND), U1.G9 (GND), U6.3 (GND), U6.7 (GND), XTAL3.1 (GND), XTAL3.4 (GND); no longer J5.26 (Pin_26), J5.27 (Pin_27), J5.28 (Pin_28), J5.29 (Pin_29), J5.30 (Pin_30), J5.56 (Pin_56), J5.57 (Pin_57), J5.58 (Pin_58), J5.59 (Pin_59), J5.60 (Pin_60), R11.2, R2.1, R3.1, R4.1, R6.1, R7.1
- net I2C2_SCL: no longer R13.1
- net I2C2_SDA: no longer R12.1
- net I2S6_CK/SPI1_SCK: now also J5.52 (Pin_52); no longer J5.12 (Pin_12)
- net I2S6_MCK: no longer J5.10 (Pin_10)
- net I2S6_SDI/SPI1_MISO: now also J5.51 (Pin_51); no longer J5.13 (Pin_13)
- net I2S6_SDO/SPI1_MOSI: no longer J5.14 (Pin_14)
- net I2S6_WS/SPI1_NSS: no longer J5.11 (Pin_11)
- net LED1: now also J5.12 (Pin_12); no longer J5.17 (Pin_17)
- net LED2: now also J5.13 (Pin_13); no longer J5.18 (Pin_18), U2.93 (PB5)
- net SDIO_CLK: now also R6.1, U1.52 (SDIO_CLK)
- net SDIO_CMD: now also R4.1, U1.51 (SDIO_CMD); no longer R25.1
- net SDMMC_CLK: now also R6.2
- net SDMMC_CMD: no longer R25.2
- net SDMMC_D0: now also R23.2, R25.2
- net SDMMC_D1: now also R13.2, R22.2; no longer R23.2
- net SDMMC_D2: now also R12.2, R21.2; no longer R22.2
- net SDMMC_D3: now also R7.2; no longer R21.2
- net STAT1: now also J5.14 (Pin_14); no longer J5.19 (Pin_19)
- net STAT2: now also J5.15 (Pin_15); no longer J5.20 (Pin_20)
- net SWCLK: now also J5.11 (Pin_11); no longer J5.52 (Pin_52)
- net SWDIO: now also J5.10 (Pin_10); no longer J5.51 (Pin_51)
- net SYS: now also J5.27 (Pin_27), J5.28 (Pin_28), J5.29 (Pin_29), J5.30 (Pin_30), J5.57 (Pin_57), J5.58 (Pin_58), J5.59 (Pin_59), J5.60 (Pin_60), U6.1 (IN), U6.2 (EN); no longer C5.1
- net USBD+: now also J5.45 (Pin_45); no longer J5.44 (Pin_44)
- net USBD-: now also J5.44 (Pin_44); no longer J5.45 (Pin_45)
- net VUSB: now also J5.31 (Pin_31), J5.32 (Pin_32), J5.33 (Pin_33), J5.34 (Pin_34), J5.35 (Pin_35), J5.36 (Pin_36), J5.37 (Pin_37), J5.38 (Pin_38); no longer C1.1, J5.1 (Pin_1), J5.2 (Pin_2), J5.3 (Pin_3), J5.4 (Pin_4), J5.5 (Pin_5), J5.6 (Pin_6), J5.7 (Pin_7), J5.8 (Pin_8)
- net WL_DEV_WAKE: now reaches U2.17 (PA1)
- net WL_DEV_WAKE: now also U1.18 (LHL_GPIO1_WL_DEV_WAKE)
- net BT_UART4_RTS: now reaches U2.66 (PA15)
- net BT_UART4_RTS: now also U1.57 (BT_UART_RTS_N)
- net BT_UART4_TX: now reaches U2.70 (PC10)
- net BT_UART4_TX: now also U1.55 (BT_UART_TXD)
- net BT_UART4_RX: now reaches U2.71 (PC11)
- net BT_UART4_RX: now also U1.56 (BT_UART_RXD)
- net BT_DEV_WAKE: now reaches U2.73 (PM0)
- net BT_DEV_WAKE: now also U1.66 (BT_DEV_WAKE)
- net BT_REG_ON: now reaches U2.80 (PM5)
- net BT_REG_ON: now also U1.63 (BT_REG_ON)
- removed net +BATT: C13.1, J5.31 (Pin_31), J5.32 (Pin_32), J5.33 (Pin_33), J5.34 (Pin_34), J5.35 (Pin_35), J5.36 (Pin_36), J5.37 (Pin_37), J5.38 (Pin_38)
- net EN_3V3REG: no longer names the net of U2.74 (PM1)
- net JTAG_TCK: no longer names the net of J5.47 (Pin_47)
- net JTAG_TDI: no longer names the net of J5.49 (Pin_49)
- net JTAG_TDO: no longer names the net of J5.48 (Pin_48)
- net JTAG_TMS: no longer names the net of J5.46 (Pin_46)
- new net: PGLED1.1 (K), U6.4 (PG)
- new net: PGLED1.2 (A), R11.2
- new net: PGLED2.1 (K), R10.1
- new net BT_INTERFACE_SELECT: R2.1, U1.65 (GPIO_12)
- new net BT_UART4_CTS: U1.54 (BT_UART_CTS_N), U2.26 (PB0)
- new net SDIO_DATA0: R25.1, U1.50 (SDIO_DATA0)
- new net SDIO_DATA1: R13.1, U1.49 (SDIO_DATA1)
- new net SDIO_DATA2: R12.1, U1.48 (SDIO_DATA2)
- new net SDIO_DATA3: R7.1, U1.47 (SDIO_DATA3)
- new net SDIO_SELECT: R3.1, U1.24 (GPIO_1)
- new net WL_REG_ON: U1.28 (WL_REG_ON), U2.93 (PB5)
- new net WiFi_OSC32: U1.27 (LPOIN), XTAL3.2 (CLK_OUT)
- no-connect marks 105 -> 46
Other:
- note added: "3.3V - Aux Regulator (WiFi module) TBR"
- note added: "Antenna Pins, unused for MH4 module"
- note added: "BT Interface Select (UART)"
- note added: "Strapping Option for SDIO"
- note added: "WiFi Module - Sona IF573 2x2 WiFi 6E Module"
- note added: "YELLOW LED == Connected to Wifi"
- note removed: "3.3V - Aux Regulator (for IRIS W106)"
- note removed: "BLUE LED == Connected to Wifi"
- note removed: "CHARGER CONFIGURATION"
- note removed: "Charger+PowerPath BQ25185"
- note removed: "Connect 10k resistor not using TRM"
- note removed: "FUEL GAUGE"
- note removed: "JST Connector for battery"
- note removed: "STATUS LED"
- note removed: "Set Charge Voltage to 4.2V, Input limit to 1.1A"
- note removed: "USB C CONNECTOR"
- note removed: "WiFi Coprocessor - Iris W106"

Commit message: added back USB connector, added power path manager, went with smaller connector
Parts:
- removed J5: CONN_MEZANNINE, ENCHANTI_connectors:CON_536250674_MOL, symbol ENCHANTI_connectors:Module_Connector
- removed SYS2: SYS, symbol power-symbols:VSYS
- added C23: 0.1uF, Capacitor_SMD:C_0402_1005Metric, symbol Device:C
- added J1: 878-22-004-10-011101, ENCHANTI_connectors:CONN_878-22-004-10-011101_MIM, symbol ENCHANTI_connectors:878-22-004-10-011101
- added J3: USB_C_Receptacle_USB2.0, Connector_USB:USB_C_Receptacle_GCT_USB4105-xx-A_16P_TopMnt_Horizontal, symbol Connector:USB_C_Receptacle_USB2.0
- added R24, R26: 5k1, Resistor_SMD:R_0402_1005Metric, symbol Device:R_US
- added U5: USBLC6-2P6, Package_TO_SOT_SMD:SOT-666, symbol Power_Protection:USBLC6-2P6
- added U7: LM66200DRLR, ENCHANTI_regulators:SOT-5X3_DRL_TEX, symbol ENCHANTI_regulators:LM66200DRLR
Connections:
- net CAN_H: now also J1.2
- net CAN_L: now also J1.3
- net GND: now also C23.2, J1.4, J3.A1 (GND), J3.A12 (GND), J3.B1 (GND), J3.B12 (GND), J3.S1 (SHIELD), R24.1, R26.1, U5.2 (GND)
- net SYS: now also J1.1
- net USBD+: now also U5.4 (I/O2)
- net USBD-: now also U5.6 (I/O1)
- net VUSB: now also C23.1, J3.A4 (VBUS), J3.A9 (VBUS), J3.B4 (VBUS), J3.B9 (VBUS), U5.5 (VBUS)
- net ANG2: no longer names the net of U2.27 (PB1)
- net ANG3: no longer names the net of U2.28 (PB2)
- net BTN1: no longer names the net of U2.99 (PB8)
- net BTN2: no longer names the net of U2.100 (PB9)
- net FSR1: no longer names the net of U2.83 (PM8)
- net FSR2: no longer names the net of U2.81 (PM6)
- net LED1: no longer names the net of U2.2 (PC13)
- net LED2: no longer names the net of U2.60 (PA9)
- new net: J3.A5 (CC1), R26.2
- new net: J3.B5 (CC2), R24.2
- new net D+: J3.A6 (D+), J3.B6 (D+), U5.3 (I/O2)
- new net D-: J3.A7 (D-), J3.B7 (D-), U5.1 (I/O1)
- no-connect marks 46 -> 54
Other:
- note added: "Magnetic Spring-loaded header"
- note added: "USB C CONNECTOR + POWER PATH"
- note removed: "Mezannine Connector"

Commit message: removed unused nets, simplified connector
Parts:
- removed J1: 878-22-004-10-011101, ENCHANTI_connectors:CONN_878-22-004-10-011101_MIM, symbol ENCHANTI_connectors:878-22-004-10-011101
- removed R15, R16: 1k, Resistor_SMD:R_0402_1005Metric, symbol Device:R_US
- removed STATLED1: GENERAL STATUS, LED_SMD:LED_0402_1005Metric, symbol Device:LED
- removed STATLED2: WIFISTATUS, LED_SMD:LED_0402_1005Metric, symbol Device:LED
- removed SYS3: SYS, symbol power-symbols:VSYS
- added J1: Enchanti-Module-Receptacle, ENCHANTI_connectors:Enchanti-Module-Receptacle, symbol ENCHANTI_connectors:Enchanti-Module-Receptacle
- added R27: 10k, Resistor_SMD:R_0402_1005Metric, symbol Device:R_US
- added SYS2: SYS, symbol power-symbols:VSYS
- U6: footprint ENCHANTI_regulators:NCV8187AMT330TAG_ONS -> ENCHANTI_regulators:NCV8187AMT330TAG_ONS-L
Connections:
- net CAN_H: now also J1.3 (CANL)
- net CAN_L: now also J1.2 (CANH)
- net GND: now also U7.1 (GND), U7.4 (ON), U7.5 (GND), J1.4 (GND)
- net SYS: now also U7.2 (VOUT), U7.7 (VOUT), SYS2.1 (SYS)
- net VUSB: now also U7.6 (VIN2)
- net +5V: now reaches U7.3 (VIN1)
- net +5V: now also J1.1 (VSYS), R27.1
- net at U7.8 (ST): now also R27.2
- net INT_LEDB: no longer names the net of U2.75 (PM2)
- net INT_LEDO: no longer names the net of U2.76 (PM3)
- no-connect marks 54 -> 56
Other:
- note removed: "ORANGE LED == Setting up/Fail State"
- note removed: "YELLOW LED == Connected to Wifi"

Commit message: added components to 2S battery charger, changing up the enchanti module design
Parts:
- removed J3: USB_C_Receptacle_USB2.0, Connector_USB:USB_C_Receptacle_GCT_USB4105-xx-A_16P_TopMnt_Horizontal, symbol Connector:USB_C_Receptacle_USB2.0
- added J3: USB4105-GF-A, Connector_USB:USB_C_Receptacle_GCT_USB4105-xx-A_16P_TopMnt_Horizontal, symbol ENCHANTI_connectors:USB4105-GF-A
- added U11: STM32H562RITx, Package_QFP:LQFP-64_10x10mm_P0.5mm, symbol MCU_ST_STM32H5:STM32H562RITx
Connections:
- net D+: now also J3.A6 (D+), J3.B6 (D+)
- net D-: now also J3.A7 (D-), J3.B7 (D-)
- net GND: now also J3.A1 (GND), J3.A12 (GND), J3.B1 (GND), J3.B12 (GND), J3.S1 (SHIELD)
- net VUSB: now also J3.A4 (VBUS), J3.A9 (VBUS), J3.B4 (VBUS), J3.B9 (VBUS)
- net at R26.2: now also J3.A5 (CC1)
- net at R24.2: now also J3.B5 (CC2)
- new net: U11.18 (VSS), U11.31 (VSS), U11.47 (VSS), U11.63 (VSS)
Other:
- note added: "1.8V main regulator (for MCU Power)"
- note added: "Battery Connector"
- note added: "Connector to external systems"
- note added: "HSE (swap to crystal resonator for lower power consumption)"
- note added: "NEEDS - BATT+ - GND - SDA - SCL"
- note added: "STM32H562 (APPLICATION MCU)"
- note added: "STM32H7R3 (WIFI MCU)"
- note added: "SWITCH TO M2 module and footprint"
- note removed: "1.8V main regulator (for STM32H7R3)"
- note removed: "HSE (24MHz)"
- note removed: "Magnetic Spring-loaded header"
- note removed: "STM32H7R3"
- moved on the sheet: C10, C11, C12, C14, C15, C16, C17, C18, C19, C2, C20, C21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

Commit message: Revert "added components to 2S battery charger, changing up the enchanti module design"
This reverts commit 22a1e749752c1cc608d102de7de6baf7b482e290.
Parts:
- removed J3: USB4105-GF-A, Connector_USB:USB_C_Receptacle_GCT_USB4105-xx-A_16P_TopMnt_Horizontal, symbol ENCHANTI_connectors:USB4105-GF-A
- removed U11: STM32H562RITx, Package_QFP:LQFP-64_10x10mm_P0.5mm, symbol MCU_ST_STM32H5:STM32H562RITx
- added J3: USB_C_Receptacle_USB2.0, Connector_USB:USB_C_Receptacle_GCT_USB4105-xx-A_16P_TopMnt_Horizontal, symbol Connector:USB_C_Receptacle_USB2.0
Connections:
- net D+: now also J3.A6 (D+), J3.B6 (D+)
- net D-: now also J3.A7 (D-), J3.B7 (D-)
- net GND: now also J3.A1 (GND), J3.A12 (GND), J3.B1 (GND), J3.B12 (GND), J3.S1 (SHIELD)
- net VUSB: now also J3.A4 (VBUS), J3.A9 (VBUS), J3.B4 (VBUS), J3.B9 (VBUS)
- net at R26.2: now also J3.A5 (CC1)
- net at R24.2: now also J3.B5 (CC2)
Other:
- note added: "1.8V main regulator (for STM32H7R3)"
- note added: "HSE (24MHz)"
- note added: "Magnetic Spring-loaded header"
- note added: "STM32H7R3"
- note removed: "1.8V main regulator (for MCU Power)"
- note removed: "Battery Connector"
- note removed: "Connector to external systems"
- note removed: "HSE (swap to crystal resonator for lower power consumption)"
- note removed: "NEEDS - BATT+ - GND - SDA - SCL"
- note removed: "STM32H562 (APPLICATION MCU)"
- note removed: "STM32H7R3 (WIFI MCU)"
- note removed: "SWITCH TO M2 module and footprint"
- moved on the sheet: C10, C11, C12, C14, C15, C16, C17, C18, C19, C2, C20, C21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
