File: enchantiS3-board/enchantiS3.kicad_sch (KiCad schematic)
At the start: 68 parts, among them J1 USB_C_Receptacle_USB2.0, J2 Conn_01x03_MountingPin, SW1 B3U-1000P, SW2 B3U-1000P, U1 USBLC6-2P6, U2 MCP73871, U3 NCP167AMX330TBG, U5 NCP167AMX330TBG, U6 MAX17262REWL+T, U7 LSM6DSV16XTR, U8 IIS2MDCTR, U9 TJA1051TK-3

Commit message: changed color of board for 3D viewer
Parts:
- removed R20: 2k, Resistor_SMD:R_0402_1005Metric, symbol Device:R_US
- removed TH1: 10k, Resistor_SMD:R_0402_1005Metric, symbol Device:Thermistor_NTC_US
- removed TP1: TestPoint, TestPoint:TestPoint_Pad_D1.0mm, symbol Connector:TestPoint
- added R11: 1k, Resistor_SMD:R_0402_1005Metric, symbol Device:R_US
- added R14: 10k, Resistor_SMD:R_0402_1005Metric, symbol Device:R_US
Connections:
- net CHRG+: now also BOARDLAYOUT1.3.3 (CHARG+)
- net GND: now also BOARDLAYOUT1.3.4 (GND), R11.1, R14.2; no longer BOARDLAYOUT1.3.3 (GND)
- net PROG1: now also R11.2
- net THRM: now also R14.1

Commit message: switched battery charged and regulators
Parts:
- removed C14: 10uF, Capacitor_SMD:C_0603_1608Metric, symbol Device:C
- removed C16, C17: 1uF, Capacitor_SMD:C_0402_1005Metric, symbol Device:C
- removed CHARGLED3: PG, LED_SMD:LED_0402_1005Metric, symbol Device:LED
- removed R11, R24: 1k, Resistor_SMD:R_0402_1005Metric, symbol Device:R_US
- removed R17: 24.9k, Resistor_SMD:R_0402_1005Metric, symbol Device:R_US
- removed R18: 330k, Resistor_SMD:R_0402_1005Metric, symbol Device:R_US
- removed R4: 110k, Resistor_SMD:R_0402_1005Metric, symbol Device:R_US
- removed R9: 10k, Resistor_SMD:R_0402_1005Metric, symbol Device:R_US
- removed SYS1, SYS3, SYS5: SYS, symbol power-symbols:VSYS
- removed U2: MCP73871, Package_DFN_QFN:QFN-20-1EP_4x4mm_P0.5mm_EP2.5x2.5mm, symbol Battery_Management:MCP73871
- removed U3, U5: NCP167AMX330TBG, XDFN4_1X1_711AJ_ONS, symbol NCP167AMX330TBG:NCP167AMX330TBG
- removed U9: TJA1051TK-3, Package_DFN_QFN:DFN-8-1EP_3x3mm_P0.65mm_EP1.55x2.4mm, symbol Interface_CAN_LIN:TJA1051TK-3
- added C11, C12, C22: 1uF, Capacitor_SMD:C_0402_1005Metric, symbol Device:C
- added C21, C23: 10uF, Capacitor_SMD:C_0603_1608Metric, symbol Device:C
- added R19: 0.43k, Resistor_SMD:R_0402_1005Metric, symbol Device:R_US
- added R20: 13k, Resistor_SMD:R_0402_1005Metric, symbol Device:R_US
- added R21: 10k, Resistor_SMD:R_0402_1005Metric, symbol Device:R_US
- added SYS6, SYS7, SYS8: SYS, symbol power-symbols:VSYS
- added TP1: TestPoint, TestPoint:TestPoint_Pad_D1.0mm, symbol Connector:TestPoint
- added U10: BQ25185DLHR, BQ25185-footprints:WSON10_DLH_TEX-M, symbol BQ25185:BQ25185DLHR
- added U2: PTCAN3413DRBR, TCAN3413-footprints:VSON8-DRB_TEX, symbol TCAN3413:PTCAN3413DRBR
- added U3, U4: NCV8187AMT330TAG, NCV8187-footprints:NCV8187AMT330TAG_ONS-L, symbol NCV8187:NCV8187AMT330TAG
- C3: value 4.7uF -> 1uF; footprint Capacitor_SMD:C_0603_1608Metric -> Capacitor_SMD:C_0402_1005Metric; Description Value Pkg 4.7 µF ±10% 16V Ceramic Capacitor X5R 0603 (1608 Metric) -> 1 µF ±10% 16V Ceramic Capacitor X5R 0402 (1005 Metric); Mfg Part # CL10A475KO8NNNC -> CL05A105KO5NNNC; mpn CL10A475KO8NNNC -> CL05A105KO5NNNC
- C8: value 4.7uF -> 0.1uF; footprint Capacitor_SMD:C_0603_1608Metric -> Capacitor_SMD:C_0402_1005Metric; Description Value Pkg 4.7 µF ±10% 16V Ceramic Capacitor X5R 0603 (1608 Metric) -> 0.1 µF ±10% 16V Ceramic Capacitor X7R 0402 (1005 Metric); Mfg Part # CL10A475KO8NNNC -> CL05B104KO5NNNC; mpn CL10A475KO8NNNC -> CL05B104KO5NNNC
Connections:
- net IO38 is gone; now on net MAG_INT: MCU1.31 (GPIO38/FSPIWP/SUBSPIWP)
- net +3V3: now also BOARDLAYOUT1.3.3 (3v3), C3.1, C8.1, C12.1, U2.3 (VCC), U2.5 (VIO), U4.5 (SNS), U4.6 (OUT); no longer C5.1, U8.3 (CS)
- net 3V3_AUX: now also C5.1, U3.5 (SNS), U3.6 (OUT)
- net CAN_H: now also U2.7 (CANH)
- net CAN_L: now also U2.6 (CANL)
- net CAN_MODE: now also U2.8 (STB)
- net CAN_RX: now also U2.4 (RXD)
- net CAN_TX: now also U2.1 (TXD)
- net CHRG+: now also C22.1, TP1.1, U10.2 (BAT); no longer BOARDLAYOUT1.3.3 (CHARG+), C8.1
- net GND: now also C11.2, C12.2, C21.2, C22.2, C23.2, R19.1, R20.1, R21.1, U10.11 (EPAD), U10.4 (/CE), U10.5 (GND), U2.2 (GND), U2.9 (THERMAL_PAD), U3.3 (GND), U3.7 (GND), U4.3 (GND), U4.7 (GND)
- net LDO_EN: now also U3.2 (EN)
- net STAT2: now also U10.3 (STAT2)
- net SYS: now also C11.1, C23.1, SYS6.1 (SYS), SYS7.1 (SYS), SYS8.1 (SYS), U10.1 (SYS), U3.1 (IN), U4.1 (IN), U4.2 (EN); no longer C3.1
- net VUSB: now also C21.1, U10.10 (IN)
- net MAG_INT: now reaches U8.7 (INT/DRDY)
- net IO15 renamed BLUELED
- net IO16 renamed ORANGELED
- net IO17 renamed SPC
- net SPC: now also U8.1 (SCL/SPC)
- net IO18 renamed SDIO
- net SDIO: now also U8.4 (SDA/SDI/SDO)
- net IO45 renamed CS1
- net CS1: now also U8.3 (CS)
- net IO7 renamed FSR2
- net IO8 renamed FSR1
- net IO9 renamed BTN
- net SCL_EXT: no longer names the net of U7.3 (SCx/AH2/QVAR2)
- net SCL_EXT: no longer U8.1 (SCL/SPC)
- net SDA_EXT: no longer names the net of U7.2 (SDx/AH1/QVAR1)
- net SDA_EXT: no longer U8.4 (SDA/SDI/SDO)
- net STAT renamed STAT1
- net STAT1: now also U10.9 (STAT1)
- new net ISET: R19.2, U10.8 (ISET)
- new net TMR: R21.2, U10.6 (TS/MR)
- new net VSET: R20.2, U10.7 (ILIM/VSET)
- no-connect marks 8 -> 11
Other:
- note added: "Charger+PowerPath BQ25185"
- note removed: "Charge Limit 2kOhm = 500mA"
- note removed: "Charge Termincation Current 24.9koHm = 40mA charge termination"
- note removed: "Charger+PowerPath MCP73871"
- note removed: "Voltage Charge Control"
- moved on the sheet: BT1, R22, R3

Commit message: Updated BOM and manufacturing files, removed CAN transceiver, updated silkscreen
Parts:
- removed C3: 1uF, Capacitor_SMD:C_0402_1005Metric, symbol Device:C
- removed C8: 0.1uF, Capacitor_SMD:C_0402_1005Metric, symbol Device:C
- removed J2: Conn_01x03_MountingPin, Connector_JST:JST_PH_B3B-PH-SM4-TB_1x03-1MP_P2.00mm_Vertical, symbol Connector_Generic_MountingPin:Conn_01x03_MountingPin
- removed U2: PTCAN3413DRBR, TCAN3413-footprints:VSON8-DRB_TEX, symbol TCAN3413:PTCAN3413DRBR
- added TOUCH2: JST-SH-1x04 1.0mm, Connector_JST:JST_SH_BM04B-SRSS-TB_1x04-1MP_P1.00mm_Vertical, symbol Connector_Generic_MountingPin:Conn_01x04_MountingPin
- R21: Description Value Pkg 1 kOhms ±1% 0.1W, 1/10W Chip Resistor 0402 (1005 Metric) Au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 -> 10 kOhms ±1% 0.1W, 1/10W Chip Resistor 0402 (1005 Metric) A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; Mfg Part # ERJ-2RKF1001X -> ERJ-2RKF1002X
- U10: Description Value Pkg (none) -> Charger IC Multi-Chemistry 10-WSON (2.2x2); Manufacturer (none) -> Texas Instruments; Mfg Part # (none) -> BQ25185DLHR
- U3, U4: Description Value Pkg (none) -> Linear Voltage Regulator IC Positive Fixed 1 Output 1.2A 6-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; Manufacturer (none) -> onsemi; Mfg Part # (none) -> NCV8187AMT330TAG
- U7: Description Value Pkg (none) -> Accelerometer, Gyroscope, Temperature, 6 Axis Sensor I2C, S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; Manufacturer (none) -> STMicroelectronics; Mfg Part # (none) -> LSM6DSV16XTR
- U8: Description Value Pkg (none) -> Magnetoresistive Sensor X, Y, Z Axis 12-LGA (2x2); Manufacturer (none) -> STMicroelectronics; Mfg Part # (none) -> IIS2MDCTR
Connections:
- net IO4 is gone; now on net CS1: MCU1.4 (GPIO4/TOUCH4/ADC1_CH3)
- net CS1: no longer MCU1.35 (MTMS/GPIO42)
- net GND: now also TOUCH2.MP (MountPin)
- net CAN_MODE renamed EVT4
- net EVT4: now also TOUCH2.4 (Pin_4)
- net CAN_RX renamed EVT2
- net EVT2: now also TOUCH2.2 (Pin_2)
- net CAN_TX renamed EVT1
- net EVT1: now also TOUCH2.1 (Pin_1)
- new net EVT3: MCU1.35 (MTMS/GPIO42), TOUCH2.3 (Pin_3)
Other:
- note added: "Connect to MCU"
- note added: "GPIO"
- note added: "Interrupt Signals from touch board"
- note removed: "3 pin JST-PH3 connector for CAN-FD connection to touch boards"
- note removed: "CAN Transreceiver"
- moved on the sheet: R12, R13, TOUCH1

Commit message: fix incorrect capacitor value in BOM
Parts:
- C13, C21, C23: Mfg Part # CL10A105KO8NNNC -> CL10A106KO8NNNC
Changed lines of the file:
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@@
       (effects (font (size 1.27 1.27)) hide)
     )
-    (property "Mfg Part #" "CL10A105KO8NNNC" (at 26.035 135.255 0)
+    (property "Mfg Part #" "CL10A106KO8NNNC" (at 26.035 135.255 0)
       (effects (font (size 1.27 1.27)) hide)
     )
@@
       (effects (font (size 1.27 1.27)) hide)
     )
-    (property "Mfg Part #" "CL10A105KO8NNNC" (at 121.92 39.37 0)
+    (property "Mfg Part #" "CL10A106KO8NNNC" (at 121.92 39.37 0)
       (effects (font (size 1.27 1.27)) hide)
     )
@@
       (effects (font (size 1.27 1.27)) hide)
     )
-    (property "Mfg Part #" "CL10A105KO8NNNC" (at 48.895 135.255 0)
+    (property "Mfg Part #" "CL10A106KO8NNNC" (at 48.895 135.255 0)
       (effects (font (size 1.27 1.27)) hide)
     )

Commit message: updated pullup resistors to 10k
Parts:
- R1, R2: value 1k -> 10k; Description Value Pkg 1 kOhms ±1% 0.1W, 1/10W Chip Resistor 0402 (1005 Metric) Au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 -> 10 kOhms ±1% 0.1W, 1/10W Chip Resistor 0402 (1005 Metric) A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; Mfg Part # ERJ-2RKF1001X -> ERJ-2RKF1002X
Changed lines of the file:
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@@
   (symbol (lib_id "Device:R_US") (at 390.525 209.55 0) (unit 1)
     (in_bom yes) (on_board yes) (dnp no)
-    (property "Reference" "R2" (at 386.715 208.28 0)
+    (property "Reference" "R2" (at 385.445 208.28 0)
       (effects (font (size 1.27 1.27)) (justify left))
     )
-    (property "Value" "1k" (at 386.715 210.82 0)
+    (property "Value" "10k" (at 385.445 210.82 0)
       (effects (font (size 1.27 1.27)) (justify left))
     )
@@
       (effects (font (size 1.27 1.27)) hide)
     )
-    (property "Description Value Pkg" "1 kOhms ±1% 0.1W, 1/10W Chip Resistor 0402 (1005 Metric) Automotive AEC-Q200 Thick Film" (at 390.525 209.55 0)
+    (property "Description Value Pkg" "10 kOhms ±1% 0.1W, 1/10W Chip Resistor 0402 (1005 Metric) Automotive AEC-Q200 Thick Film" (at 390.525 209.55 0)
       (effects (font (size 1.27 1.27)) hide)
     )
-    (property "Mfg Part #" "ERJ-2RKF1001X" (at 390.525 209.55 0)
+    (property "Mfg Part #" "ERJ-2RKF1002X" (at 390.525 209.55 0)
       (effects (font (size 1.27 1.27)) hide)
     )
@@
   (symbol (lib_id "Device:R_US") (at 367.665 208.915 0) (unit 1)
     (in_bom yes) (on_board yes) (dnp no)
-    (property "Reference" "R1" (at 363.855 207.645 0)
+    (property "Reference" "R1" (at 362.585 207.645 0)
       (effects (font (size 1.27 1.27)) (justify left))
     )
-    (property "Value" "1k" (at 363.855 210.185 0)
+    (property "Value" "10k" (at 362.585 210.185 0)
       (effects (font (size 1.27 1.27)) (justify left))
     )
@@
       (effects (font (size 1.27 1.27)) hide)
     )
-    (property "Description Value Pkg" "1 kOhms ±1% 0.1W, 1/10W Chip Resistor 0402 (1005 Metric) Automotive AEC-Q200 Thick Film" (at 367.665 208.915 0)
+    (property "Description Value Pkg" "10 kOhms ±1% 0.1W, 1/10W Chip Resistor 0402 (1005 Metric) Automotive AEC-Q200 Thick Film" (at 367.665 208.915 0)
       (effects (font (size 1.27 1.27)) hide)
     )
-    (property "Mfg Part #" "ERJ-2RKF1001X" (at 367.665 208.915 0)
+    (property "Mfg Part #" "ERJ-2RKF1002X" (at 367.665 208.915 0)
       (effects (font (size 1.27 1.27)) hide)
     )

Commit message: finsished routing for revision 4 of enchantiS3, finished routing for  enchantiS3 Touch
Parts:
- removed C10: 1uF, Capacitor_SMD:C_0402_1005Metric, symbol Device:C
- removed C18: 220nF, Capacitor_SMD:C_0402_1005Metric, symbol Device:C
- removed C7: 0.1uF, Capacitor_SMD:C_0402_1005Metric, symbol Device:C
- removed CHARGLED2: S2, LED_SMD:LED_0402_1005Metric, symbol Device:LED
- removed R22: 1k, Resistor_SMD:R_0402_1005Metric, symbol Device:R_US
- removed U3, U4: NCV8187AMT330TAG, NCV8187-footprints:NCV8187AMT330TAG_ONS-L, symbol NCV8187:NCV8187AMT330TAG
- removed U8: IIS2MDCTR, LGA-12_2X2X0P7_STM, symbol IIS2MDCTR:IIS2MDCTR
- added C3: 220nF, Capacitor_SMD:C_0402_1005Metric, symbol Device:C
- added R4, R9: 2k2, Resistor_SMD:R_0402_1005Metric, symbol Device:R_US
- added U2: MMC5633NJL, Package_BGA:WLP-4_0.86x0.86mm_P0.4mm, symbol Sensor_Magnetic:MMC5633NJL
- added U5, U8: NCP167AMX330TBG, XDFN4_1X1_711AJ_ONS, symbol NCP167:NCP167AMX330TBG
- FP1: renamed from TOUCH2; footprint Connector_JST:JST_SH_BM04B-SRSS-TB_1x04-1MP_P1.00mm_Vertical -> Connector_JST:JST_SH_BM06B-SRSS-TB_1x06-1MP_P1.00mm_Vertical; symbol Connector_Generic_MountingPin:Conn_01x04_MountingPin -> Connector_Generic_MountingPin:Conn_01x06_MountingPin; Mfg Part # BM04B-SRSS-TB -> BM06B-SRSS-TB
- R3: value 1k -> 2k2; Description Value Pkg 1 kOhms ±1% 0.1W, 1/10W Chip Resistor 0402 (1005 Metric) Au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 -> 2.2 kOhms ±1% 0.1W, 1/10W Chip Resistor 0402 (1005 Metric) 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; Mfg Part # ERJ-2RKF1001X -> ERJ-2RKF2201X; mpn ERJ-2RKF1001X -> ERJ-2RKF2201X
Connections:
- net MAG_INT is gone; now on net BTN_FP: MCU1.31 (GPIO38/FSPIWP/SUBSPIWP)
- net +3V3: now also C3.1, R4.2, R9.2, U2.B1 (VDD), U5.1 (OUT)
- net 3V3_AUX: now also FP1.1 (Pin_1), U8.1 (OUT)
- net GND: now also R3.2, C3.2, U2.A1 (VSA), U5.2 (GND), U5.5 (GND), U8.2 (GND), U8.5 (GND)
- net LDO_EN: now also U8.3 (EN)
- net STAT1: now also FP1.6 (Pin_6); no longer R3.2
- net STAT2: now also FP1.5 (Pin_5)
- net SYS: now also U5.3 (EN), U5.4 (IN), U8.4 (IN)
- net CS1: no longer names the net of MCU1.4 (GPIO4/TOUCH4/ADC1_CH3)
- net EVT1 renamed LED1
- net LED1: now also FP1.3 (Pin_3); no longer FP1.1 (Pin_1)
- net EVT2 renamed BTN_FP
- net BTN_FP: no longer MCU1.34 (MTDI/GPIO41/CLK_OUT1)
- net EVT3 renamed LED3
- net LED3: no longer FP1.3 (Pin_3)
- net EVT4 renamed LED2
- net LED2: now also MCU1.34 (MTDI/GPIO41/CLK_OUT1); no longer MCU1.24 (GPIO47/SPICLK_P/SUBSPICLK_P_DIFF)
- net SDIO renamed SDA2
- net SDA2: now also R9.1, U2.B2 (SDA)
- net SPC renamed SCL2
- net SCL2: now also R4.1, U2.A2 (SCL)
- new net LED4: MCU1.24 (GPIO47/SPICLK_P/SUBSPICLK_P_DIFF)
Other:
- note added: "Connect to Frontplate"
- note added: "Front Plate Conntector"
- note removed: "Connect to MCU"
- note removed: "GPIO"
- note removed: "Interrupt Signals from touch board"
- note removed: "Table 5.1 in MCP73871 Datasheet shows table for status outputs"
- moved on the sheet: C12, C4, C5

Commit message: updated project to kicad 8.0, switched to using enchantiLibrary footprint/symbols, switched connectors to molex picoclasp, updated imu
Parts:
- removed C1, C20: 0.1uF, Capacitor_SMD:C_0402_1005Metric, symbol Device:C
- removed C2: 0.47uF, Capacitor_SMD:C_0402_1005Metric, symbol Device:C
- removed C6: 1uF, Capacitor_SMD:C_0402_1005Metric, symbol Device:C
- removed R14: 10k, Resistor_SMD:R_0402_1005Metric, symbol Device:R_US
- removed R19: 0.43k, Resistor_SMD:R_0402_1005Metric, symbol Device:R_US
- removed R20: 13k, Resistor_SMD:R_0402_1005Metric, symbol Device:R_US
- removed SYS7: SYS, symbol power-symbols:VSYS
- removed TOUCH1: JST-SH-1x04 1.0mm, Connector_JST:JST_SH_BM04B-SRSS-TB_1x04-1MP_P1.00mm_Vertical, symbol Connector_Generic_MountingPin:Conn_01x04_MountingPin
- removed U10: BQ25185DLHR, BQ25185-footprints:WSON10_DLH_TEX-M, symbol BQ25185:BQ25185DLHR
- removed U5, U8: NCP167AMX330TBG, XDFN4_1X1_711AJ_ONS, symbol NCP167:NCP167AMX330TBG
- removed U6: MAX17262REWL+T, max17262-footprints:21-100221A_W91G1&plus_3_MXM, symbol max17262:MAX17262REWL+T
- removed U7: LSM6DSV16XTR, LSM6DSV16XTR-footprints:LGA14L_LSM6_STM, symbol LSM6DSV16XTR:LSM6DSV16XTR
- added C17: 1uF, Capacitor_SMD:C_0402_1005Metric, symbol Device:C
- added C18, C7: 0.1uF, Capacitor_SMD:C_0402_1005Metric, symbol Device:C
- added C8: 0.47uF, Capacitor_SMD:C_0402_1005Metric, symbol Device:C
- added H3: MountingHole, MountingHole:MountingHole_2.2mm_M2, symbol Mechanical:MountingHole
- added R11: 13k, Resistor_SMD:R_0402_1005Metric, symbol Device:R_US
- added R15: 0.3k, Resistor_SMD:R_0402_1005Metric, symbol Device:R_US
- added SYS1: SYS, symbol power-symbols:VSYS
- added TOUCH1: JST-SH-1x04 1.0mm, ENCHANTI_connectors:JST_SMD_1.0mm-4_Vertical, symbol ENCHANTI_connectors:QWIIC-CONNECTOR
- added U11: MAX17262REWL+T, ENCHANTI_battery-management:MAX17262, symbol ENCHANTI_battery-management:MAX17262REWL+T
- added U12: BQ25185DLHR, ENCHANTI_battery-management:WSON10_DLH_TEX, symbol ENCHANTI_battery-management:BQ25185DLHR
- added U13: ICM-42670-P, ENCHANTI_MEMS:LGA14_2P5X3X0P91_TDK, symbol ENCHANTI_mems:ICM-42670-P
- added U4, U9: NCP167AMX330TBG, ENCHANTI_regulators:XDFN4_1X1_711AJ_ONS, symbol ENCHANTI_regulators:NCP167AMX330TBG
- ANG1, ANG2, ANG3: value JST-SH-1.00mm 1x2 -> CONN HEADER SMD 2POS 1MM; footprint Connector_JST:JST_SH_BM02B-SRSS-TB_1x02-1MP_P1.00mm_Vertical -> ENCHANTI_connectors:Molex_Pico-Clasp_2pin_Vertical; symbol Connector_Generic_MountingPin:Conn_01x02_MountingPin -> ENCHANTI_connectors:PicoClasp_2pin; Description Value Pkg Connector Header Surface Mount 2 position 0.039" (1.00mm) -> (none); Manufacturer JST Sales America Inc. -> Molex; Mfg Part # BM02B-SRSS-TB -> 5013310207; mpn BM02B-SRSS-TB -> (none)
- BT1: Description Value Pkg Connector Header Surface Mount, Right Angle 2 position 0.07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 -> (none)
- C11, C12, C22, C4, C5, C9: Description Value Pkg 1 µF ±10% 16V Ceramic Capacitor X5R 0402 (1005 Metric) -> (none)
- C13, C21, C23: Description Value Pkg 10 µF ±10% 6.3V Ceramic Capacitor X5R 0603 (1608 Metric) -> (none)
- C15, C19: Description Value Pkg 0.1 µF ±10% 16V Ceramic Capacitor X7R 0402 (1005 Metric) -> (none)
- C3: Description Value Pkg 0.22 µF ±10% 16V Ceramic Capacitor X7R 0402 (1005 Metric) -> (none)
- CHARGLED1: Description Value Pkg Red 630nm LED Indication - Discrete 1.95V 0402 (1005 Metric) -> (none)
- FP1: value JST-SH-1x04 1.0mm -> CONN HEADER SMD 6POS 1MM; footprint Connector_JST:JST_SH_BM06B-SRSS-TB_1x06-1MP_P1.00mm_Vertical -> ENCHANTI_connectors:Molex_Pico-Clasp_501331-0607_1x06-1MP_P1.00mm_Vertical; Description Value Pkg Connector Header Surface Mount 4 position 0.039" (1.00mm) -> (none); Manufacturer JST Sales America Inc. -> Molex; Mfg Part # BM06B-SRSS-TB -> 5013310607; mpn BM04B-SRSS-TB -> (none)
- H1, H2: footprint MountingHole:MountingHole_3.2mm_M3_DIN965 -> MountingHole:MountingHole_2.2mm_M2
- J1: Description Value Pkg USB-C (USB TYPE-C) USB 2.0 Receptacle Connector 24 (16+8 Du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 -> (none)
- MCU1: Description Value Pkg Bluetooth, WiFi 802.11b/g/n, Bluetooth v5.0 Transceiver Mod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 -> (none)
- R1, R2, R21, R5: Description Value Pkg 10 kOhms ±1% 0.1W, 1/10W Chip Resistor 0402 (1005 Metric) A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 -> (none)
- R10, R8: Description Value Pkg 1 kOhms ±1% 0.1W, 1/10W Chip Resistor 0402 (1005 Metric) Au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 -> (none)
- R12, R13, R3, R4, R9: Description Value Pkg 2.2 kOhms ±1% 0.1W, 1/10W Chip Resistor 0402 (1005 Metric) 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 -> (none)
- R6, R7: Description Value Pkg 5.1 kOhms ±1% 0.1W, 1/10W Chip Resistor 0402 (1005 Metric) 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 -> (none)
- STATLED1: Description Value Pkg Blue 467nm LED Indication - Discrete 2.9V 0402 (1005 Metric) -> (none)
- STATLED2: Description Value Pkg Amber 605nm LED Indication - Discrete 2V 0402 (1005 Metric) -> (none)
- SW1, SW2: Description Value Pkg Tactile Switch SPST-NO Top Actuated Surface Mount -> (none)
- U1: Description Value Pkg 17V Clamp 5A (8/20µs) Ipp Tvs Diode Surface Mount SOT-666 -> (none); mpn USBLC6-2P6 -> (none)
- U2: Manufacturer (none) -> Memsic; Mfg Part # (none) -> MMC5633NJL
Connections:
- net +3V3: now also FP1.1 (Pin_1), C17.1, C18.1, U13.5 (VDDIO), U13.8 (VDD), U4.1 (OUT)
- net +BATT: now also C7.1, U11.A2 (BATT)
- net 3V3_AUX: now also TOUCH1.2 (3v3), U9.1 (OUT); no longer FP1.1 (Pin_1)
- net CHRG+: now also U12.2 (BAT)
- net CIPO: now also U13.1 (AP_SDO/AP_AD0)
- net COPI: now also U13.14 (AP_SDA/AP_SDIO/AP_SDI)
- net CS: now also U13.12 (AP_CS)
- net GND: now also C17.2, C18.2, C7.2, C8.2, R11.2, R15.2, TOUCH1.1 (GND), U11.A1 (TH), U11.B2 (ALRT), U11.C3 (GND), U12.11 (EPAD), U12.4 (/CE), U12.5 (GND), U13.6 (GND), U13.7 (FSYNC), U4.2 (GND), U4.5 (GND), U9.2 (GND), U9.5 (GND)
- net IMU_INT: now also U13.4 (INT1/INT)
- net IMU_INT2: now also U13.9 (INT2)
- net ISET: now also R15.1, U12.8 (ISET)
- net LDO_EN: now also U9.3 (EN)
- net REG: now also C8.1, U11.C2 (REG)
- net SCL: now also TOUCH1.4 (SCL), U11.B1 (SCL)
- net SCLK: now also U13.13 (AP_SCL/AP_SCLK)
- net SDA: now also TOUCH1.3 (SDA), U11.C1 (SDA)
- net STAT1: now also U12.9 (STAT1)
- net STAT2: now also U12.3 (STAT2)
- net SYS: now also SYS1.1 (SYS), U12.1 (SYS), U4.3 (EN), U4.4 (IN), U9.4 (IN)
- net TMR: now also U12.6 (TS/MR)
- net VSET: now also R11.1, U12.7 (ILIM/VSET)
- net VUSB: now also U12.10 (IN)
- new net: TOUCH1.NC1 (NC), TOUCH1.NC2 (NC)
- new net +BATT_SYS: U11.B3 (SYS)
- no-connect marks 11 -> 6
Other:
- note added: "Backplate Connector"
- note removed: "CHARGER CONFIGURATION"
- note removed: "Front Plate Conntector"
- moved on the sheet: ANG1, ANG3, BT1, C11, C15, C21, C22, C23, C4, C5, J1, R1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
