File: enchantiS3-board/imu.kicad_sch (KiCad schematic)
At the start: 7 parts, among them U3 ICM-42670-P, U8 MMC5983MA

Commit message: Fixed BOM errors, removed unused Mounting Hole, added rev4 BOM
Parts:
- C19: footprint Capacitor_SMD:C_0402_1005Metric -> Capacitor_SMD:C_0603_1608Metric; Manufacturer Samsung Electro-Mechanics -> Murata Electronics; Mfg Part # CL05A106MP8NUB8 -> GRT188R61C106KE13D
Changed lines of the file:
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@@
 			)
 		)
-		(property "Footprint" "Capacitor_SMD:C_0402_1005Metric"
+		(property "Footprint" "Capacitor_SMD:C_0603_1608Metric"
 			(at 97.4852 142.24 0)
 			(effects
@@
 			)
 		)
-		(property "Description" "10 µF ±20% 10V Ceramic Capacitor X5R 0402 (1005 Metric)"
+		(property "Description" "10 µF ±10% 16V Ceramic Capacitor X5R 0603 (1608 Metric)"
 			(at 96.52 138.43 0)
 			(effects
@@
 			)
 		)
-		(property "Mfg Part #" "CL05A106MP8NUB8"
+		(property "Mfg Part #" "GRT188R61C106KE13D"
 			(at 96.52 138.43 0)
 			(effects
@@
 			)
 		)
-		(property "Manufacturer" "Samsung Electro-Mechanics"
+		(property "Manufacturer" "Murata Electronics"
 			(at 96.52 138.43 0)
 			(effects
