File: enchantiS3-board/power.kicad_sch (KiCad schematic)
At the start: 23 parts, among them SW3 SYS_RST, U2 NCP187, U7 NPM1300-QEAA-R7

Commit message: Fixed BOM errors, removed unused Mounting Hole, added rev4 BOM
Parts:
- R3, R4: Manufacturer Panasonic Electronic Components -> YAGEO; Mfg Part # ERJ-2RKF2201X -> RC0402FR-072K2L
- R6: Manufacturer Panasonic Electronic Components -> YAGEO; Mfg Part # ERJ-2RKF1002X -> RC0402FR-0710KL
- TP1: now left out of the parts list
Changed lines of the file:
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@@
 			)
 		)
-		(property "Description" "10 kOhms ±1% 0.1W, 1/10W Chip Resistor 0402 (1005 Metric) Automotive AEC-Q200 Thick Film"
+		(property "Description" "10 kOhms ±1%  0.063W, 1/16W Chip Resistor 0402 (1005 Metric)"
 			(at 236.22 38.1 0)
 			(effects
@@
 			)
 		)
-		(property "Mfg Part #" "ERJ-2RKF1002X"
+		(property "Mfg Part #" "RC0402FR-0710KL"
 			(at 236.22 38.1 0)
 			(effects
@@
 			)
 		)
-		(property "Manufacturer" "Panasonic Electronic Components"
+		(property "Manufacturer" "YAGEO"
 			(at 236.22 38.1 0)
 			(effects
@@
 		(unit 1)
 		(exclude_from_sim no)
-		(in_bom yes)
+		(in_bom no)
 		(on_board yes)
 		(dnp no)
@@
 			)
 		)
+		(property "Mfg Part #" ""
+			(at 236.22 43.18 0)
+			(effects
+				(font
+					(size 1.27 1.27)
+				)
+				(hide yes)
+			)
+		)
+		(property "Manufacturer" ""
+			(at 236.22 43.18 0)
+			(effects
+				(font
+					(size 1.27 1.27)
+				)
+				(hide yes)
+			)
+		)
 		(pin "1"
 		)
@@
 			)
 		)
-		(property "Description" "2.2 kOhms ±1% 0.1W, 1/10W Chip Resistor 0402 (1005 Metric) Automotive AEC-Q200 Thick Film"
+		(property "Description" "2.2 kOhms ±1% 0.063W, 1/16W Chip Resistor 0402 (1005 Metric)"
 			(at 81.28 124.46 0)
 			(effects
@@
 			)
 		)
-		(property "Mfg Part #" "ERJ-2RKF2201X"
+		(property "Mfg Part #" "RC0402FR-072K2L"
 			(at 81.28 124.46 0)
 			(effects
@@
 			)
 		)
-		(property "Manufacturer" "Panasonic Electronic Components"
+		(property "Manufacturer" "YAGEO"
 			(at 81.28 124.46 0)
 			(effects
@@
 			)
 		)
-		(property "Description" "2.2 kOhms ±1% 0.1W, 1/10W Chip Resistor 0402 (1005 Metric) Automotive AEC-Q200 Thick Film"
+		(property "Description" "2.2 kOhms ±1% 0.063W, 1/16W Chip Resistor 0402 (1005 Metric)"
 			(at 100.33 124.46 0)
 			(effects
@@
 			)
 		)
-		(property "Mfg Part #" "ERJ-2RKF2201X"
+		(property "Mfg Part #" "RC0402FR-072K2L"
 			(at 100.33 124.46 0)
 			(effects
@@
 			)
 		)
-		(property "Manufacturer" "Panasonic Electronic Components"
+		(property "Manufacturer" "YAGEO"
 			(at 100.33 124.46 0)
 			(effects
