File: enchantiS3-board/subschematics/mcu.kicad_sch (KiCad schematic)
At the start: 7 parts, among them SW1 BOOT, SW2 ESP_RST

Commit message: Added can transceiver circuit, finished routing power traces
Connections:
- net IO0: no longer SW1.1
- net BOOT: now reaches U4.71 (GPIO61)
- net BOOT: now also SW1.1
- no-connect marks 4 -> 6
Changed lines of the file:
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@@
 	)
 	(no_connect
-		(at 60.96 88.9)
+		(at 165.1 114.3)
+	)
+	(no_connect
+		(at 162.56 114.3)
 	)
 	(no_connect
@@
 	)
 	(no_connect
+		(at 193.04 41.91)
+	)
+	(no_connect
 		(at 60.96 91.44)
 	)
@@
 	(wire
 		(pts
+			(xy 193.04 39.37) (xy 198.12 39.37)
+		)
+		(stroke
+			(width 0)
+			(type default)
+		)
+	)
+	(wire
+		(pts
 			(xy 193.04 46.99) (xy 195.58 46.99)
 		)
@@
 			(width 0)
 			(type default)
+		)
+	)
+	(label "BOOT"
+		(at 195.58 39.37 0)
+		(effects
+			(font
+				(size 1.27 1.27)
+			)
+			(justify left bottom)
 		)
 	)
@@
 		)
 	)
-	(label "IO0"
+	(label "BOOT"
 		(at 85.09 181.61 0)
 		(effects
@@
 			)
 			(justify right)
+		)
+	)
+	(netclass_flag ""
+		(length 2.54)
+		(shape round)
+		(at 165.1 114.3 180)
+		(effects
+			(font
+				(size 1.27 1.27)
+			)
+			(justify right bottom)
+		)
+		(property "Net Class" ""
+			(at 233.68 -114.3 90)
+			(show_name no)
+			(do_not_autoplace no)
+			(effects
+				(font
+					(size 1.27 1.27)
+				)
+			)
+		)
+		(property "Component Class" "Strapping Pin"
+			(at 165.1 117.602 90)
+			(show_name no)
+			(do_not_autoplace no)
+			(effects
+				(font
+					(size 1.27 1.27)
+					(italic yes)
+				)
+				(justify right)
+			)
 		)
 	)
@@
 		(length 2.54)
 		(shape round)
-		(at 60.96 129.54 270)
+		(at 162.56 114.3 180)
 		(effects
 			(font
@@
 		)
 		(property "Net Class" ""
-			(at -167.64 60.96 0)
+			(at 231.14 -114.3 90)
 			(show_name no)
 			(do_not_autoplace no)
@@
 		)
 		(property "Component Class" "Strapping Pin"
-			(at 64.262 129.54 0)
-			(show_name no)
-			(do_not_autoplace no)
-			(effects
-				(font
-					(size 1.27 1.27)
-					(italic yes)
-				)
-				(justify left)
+			(at 162.56 117.602 90)
+			(show_name no)
+			(do_not_autoplace no)
+			(effects
+				(font
+					(size 1.27 1.27)
+					(italic yes)
+				)
+				(justify right)
 			)
 		)
@@
 		(length 2.54)
 		(shape round)
-		(at 60.96 88.9 270)
+		(at 198.12 39.37 270)
 		(effects
 			(font
@@
 		)
 		(property "Net Class" ""
-			(at -167.64 20.32 0)
+			(at -30.48 -29.21 0)
 			(show_name no)
 			(do_not_autoplace no)
@@
 		)
 		(property "Component Class" "Strapping Pin"
-			(at 64.262 88.9 0)
-			(show_name no)
-			(do_not_autoplace no)
+			(at 201.422 39.37 0)
+			(show_name no)
+			(do_not_autoplace no)
+			(effects
+				(font
+					(size 1.27 1.27)
+					(italic yes)
+				)
+				(justify left)
+			)
+		)
+	)
+	(netclass_flag ""
+		(length 2.54)
+		(shape round)
+		(at 193.04 41.91 270)
+		(effects
+			(font
+				(size 1.27 1.27)
+			)
+			(justify right bottom)
+		)
+		(property "Net Class" ""
+			(at -35.56 -26.67 0)
+			(show_name no)
+			(do_not_autoplace no)
+			(effects
+				(font
+					(size 1.27 1.27)
+				)
+			)
+		)
+		(property "Component Class" "Strapping Pin"
+			(at 196.342 41.91 0)
+			(show_name no)
+			(do_not_autoplace no)
+			(effects
+				(font
+					(size 1.27 1.27)
+					(italic yes)
+				)
+				(justify left)
+			)
+		)
+	)
+	(netclass_flag ""
+		(length 2.54)
+		(shape round)
+		(at 60.96 129.54 270)
+		(effects
+			(font
+				(size 1.27 1.27)
+			)
+			(justify right bottom)
+		)
+		(property "Net Class" ""
+			(at -167.64 60.96 0)
+			(show_name no)
+			(do_not_autoplace no)
+			(effects
+				(font
+					(size 1.27 1.27)
+				)
+			)
+		)
+		(property "Component Class" "Strapping Pin"
+			(at 64.262 129.54 0)
+			(show_name no)
+			(do_not_autoplace no)
