File: enchantiS3-board/subschematics/power.kicad_sch (KiCad schematic)
At the start: 23 parts, among them SW3 SYS_RST, U2 NCP187, U7 NPM1300-QEAA-R7

Commit message: Added circuit for magnetometer, added circuit for canfd transceiver, updated circuit for USB connector
Parts:
- removed C18: 2.2uF, Capacitor_SMD:C_0402_1005Metric, symbol Device:C
- removed C20: 0.1uF, Capacitor_SMD:C_0402_1005Metric, symbol Device:C
- removed CHARGLED4: RED_LED, LED_SMD:LED_0603_1608Metric, symbol Device:LED
- removed CHARGLED5: YELLOW_LED, LED_SMD:LED_0603_1608Metric, symbol Device:LED
- removed SW3: SYS_RST, ENCHANTI_switches:SW_SPST_PTS810, symbol ENCHANTI_switches:PTS810
- removed SYS4, SYS5: SYS, symbol power-symbols:VSYS
- removed U7: NPM1300-QEAA-R7, ENCHANTI_battery-management:QFN32_5X5_NOR, symbol ENCHANTI_battery-management:NPM1300-QEAA-R7
- added C15: 0.1uF, Capacitor_SMD:C_0402_1005Metric, symbol Device:C
- added C17: 0.47uF, Capacitor_SMD:C_0402_1005Metric, symbol Device:C
- added LED3: Yellow, LED_SMD:LED_0603_1608Metric, symbol Device:LED
- added LED4: Red, LED_SMD:LED_0603_1608Metric, symbol Device:LED
- added R14: 0.43k, Resistor_SMD:R_0402_1005Metric, symbol Device:R_US
- added R15: 10k, Resistor_SMD:R_0402_1005Metric, symbol Device:R_US
- added R17: 2k2, Resistor_SMD:R_0402_1005Metric, symbol Device:R_US
- added SYS1, SYS3: SYS, symbol power-symbols:VSYS
- added TP2: TestPoint, TestPoint:TestPoint_Pad_D1.5mm, symbol Connector:TestPoint
- added TP3, TP4, TP5: TestPoint, TestPoint:TestPoint_Pad_D1.0mm, symbol Connector:TestPoint
- added U5: BQ25185DLHR, ENCHANTI_battery-management:WSON10_DLH_TEX, symbol ENCHANTI_battery-management:BQ25185DLHR
- added U6: MAX17262REWL+T, ENCHANTI_battery-management:MAX17262, symbol ENCHANTI_battery-management:MAX17262REWL+T
- C1: Mfg Part # GRM155R61E105KA12D -> GRM155R61H105KE05D
- C4: value 1uF -> 10uF; Manufacturer Murata Electronics -> Samsung Electro-Mechanics; Mfg Part # GRM155R61E105KA12D -> CL05A106MP8NUB8
- C5: value 10uF -> 1uF; footprint Capacitor_SMD:C_0603_1608Metric -> Capacitor_SMD:C_0402_1005Metric; Mfg Part # GRT188R61C106KE13D -> GRM155R61H105KE05D
- R12: value 2k -> 13k; Mfg Part # RC0402FR-072KL -> RC0402FR-0713KL; mpn (none) -> ERJ-2RKF2201X
- R18: value 2k -> 2k2; Mfg Part # RC0402FR-072KL -> RC0402FR-072K2L; mpn (none) -> ERJ-2RKF2201X
- R3, R4: value 2k2 -> 2k; Mfg Part # RC0402FR-072K2L -> RC0402FR-072KL; mpn ERJ-2RKF2201X -> (none)
Connections:
- net SCL is gone; now on net LED0: R4.1
- net SDA is gone; now on net LED1: R3.1
- net VBUSOUT is gone; now on net SYS: C4.1
- net +3V3: now also R18.1, R17.1; no longer R3.2, R4.2
- net +BATT: now also C15.1, TP5.1, U6.A1 (TH), U6.A2 (BATT)
- net GND: now also R12.2, C15.2, C17.2, R14.2, R15.1, U5.11 (EPAD), U5.4 (~{CE}), U5.5 (GND), U6.C3 (GND)
- net LED0: now also LED4.1 (K); no longer R12.2
- net LED1: now also LED3.1 (K); no longer R18.2
- net SYS: now also LED3.2 (A), LED4.2 (A), SYS1.1 (SYS), SYS3.1 (SYS), TP3.1, U5.1 (SYS); no longer C5.1
- net VUSB: now also TP2.1, U5.10 (IN)
- net VSET: now reaches R12.1
- net VSET: now also U5.7 (ILIM/VSET)
- new net CHRG+: C5.1, TP4.1, U5.2 (BAT), U6.B3 (SYS)
- new net FG_ALRT: U6.B2 (ALRT)
- new net FG_SCL: R18.2, U6.B1 (SCL)
- new net FG_SDA: R17.2, U6.C1 (SDA)
- new net ISET: R14.1, U5.8 (ISET)
- new net REG: C17.1, U6.C2 (REG)
- new net STAT1: R3.2, U5.9 (STAT1)
- new net STAT2: R4.2, U5.3 (STAT2)
- new net TS: R15.2, U5.6 (TS/MR)
- no-connect marks 3 -> 0
Other:
- note added: "BQ25185 Battery Charger + PowerPath"
- note added: "Bypass Capacitors"
- note added: "LED For Battery charging status, Table 8.2 in BQ25185 datasheet for outputs"
- note added: "MAX17262 Fuel Gauge"
- note removed: "NPM1300 Powerpath Management + Battery Charger + Fuel Gauge + Load Switch"

Commit message: Added can transceiver circuit, finished routing power traces
Parts:
- added R19: 10k, Resistor_SMD:R_0402_1005Metric, symbol Device:R_US
Connections:
- net FG_ALRT is gone; now on net GND: U6.B2 (ALRT)
- net GND: now also R19.1; no longer U5.4 (~{CE})
- new net ~{CE}: R19.2, U5.4 (~{CE})
Changed lines of the file:
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@@
 	)
 	(junction
+		(at 49.53 66.04)
+		(diameter 0)
+		(color 0 0 0 0)
+	)
+	(junction
 		(at 58.42 39.37)
 		(diameter 0)
@@
 	)
 	(junction
+		(at 59.69 147.32)
+		(diameter 0)
+		(color 0 0 0 0)
+	)
+	(junction
 		(at 115.57 138.43)
 		(diameter 0)
@@
 	(wire
 		(pts
+			(xy 45.72 66.04) (xy 49.53 66.04)
+		)
+		(stroke
+			(width 0)
+			(type default)
+		)
+	)
+	(wire
+		(pts
 			(xy 181.61 44.45) (xy 181.61 45.72)
 		)
@@
 	(wire
 		(pts
+			(xy 49.53 83.82) (xy 49.53 87.63)
+		)
+		(stroke
+			(width 0)
+			(type default)
+		)
+	)
+	(wire
+		(pts
 			(xy 53.34 54.61) (xy 54.61 54.61)
 		)
@@
 	(wire
 		(pts
-			(xy 49.53 66.04) (xy 49.53 87.63)
+			(xy 49.53 66.04) (xy 49.53 76.2)
 		)
 		(stroke
@@
 	(wire
 		(pts
+			(xy 49.53 66.04) (xy 71.12 66.04)
+		)
+		(stroke
+			(width 0)
+			(type default)
+		)
+	)
+	(wire
+		(pts
 			(xy 93.98 140.97) (xy 104.14 140.97)
 		)
@@
 	(wire
 		(pts
+			(xy 59.69 140.97) (xy 59.69 147.32)
+		)
+		(stroke
+			(width 0)
+			(type default)
+		)
+	)
+	(wire
+		(pts
 			(xy 54.61 60.96) (xy 71.12 60.96)
 		)
@@
 	(wire
 		(pts
-			(xy 49.53 66.04) (xy 71.12 66.04)
-		)
-		(stroke
-			(width 0)
-			(type default)
-		)
-	)
-	(wire
-		(pts
 			(xy 57.15 71.12) (xy 57.15 76.2)
 		)
@@
 		)
 	)
-	(hierarchical_label "FG_ALRT"
-		(shape output)
-		(at 59.69 140.97 180)
+	(hierarchical_label "FG_SCL"
+		(shape input)
+		(at 93.98 143.51 0)
 		(effects
 			(font
 				(size 1.27 1.27)
 			)
-			(justify right)
+			(justify left)
 		)
 	)
-	(hierarchical_label "FG_SCL"
+	(hierarchical_label "~{CE}"
 		(shape input)
-		(at 93.98 143.51 0)
+		(at 45.72 66.04 180)
 		(effects
 			(font
 				(size 1.27 1.27)
 			)
-			(justify left)
+			(justify right)
 		)
 	)
@@
 					(unit 1)
 				)
+			)
+		)
+	)
+	(symbol
+		(lib_id "Device:R_US")
+		(at 49.53 80.01 180)
+		(unit 1)
+		(body_style 1)
+		(exclude_from_sim no)
+		(in_bom yes)
+		(on_board yes)
+		(in_pos_files yes)
+		(dnp no)
+		(property "Reference" "R19"
+			(at 44.45 80.01 90)
+			(show_name no)
+			(do_not_autoplace no)
+			(effects
+				(font
+					(size 1.27 1.27)
+				)
+			)
+		)
+		(property "Value" "10k"
+			(at 46.99 80.01 90)
+			(show_name no)
+			(do_not_autoplace no)
+			(effects
+				(font
+					(size 1.27 1.27)
+				)
+			)
+		)
+		(property "Footprint" "Resistor_SMD:R_0402_1005Metric"
+			(at 48.514 79.756 90)
+			(hide yes)
+			(show_name no)
+			(do_not_autoplace no)
+			(effects
+				(font
+					(size 1.27 1.27)
+				)
+			)
+		)
+		(property "Datasheet" "https://www.yageo.com/upload/media/product/products/datasheet/rchip/PYu-RC_Group_51_RoHS_L_12.pdf"
+			(at 49.53 80.01 0)
+			(hide yes)
+			(show_name no)
+			(do_not_autoplace no)
+			(effects
+				(font
+					(size 1.27 1.27)
+				)
+			)
+		)
+		(property "Description" "10 kOhms ±1% 0.063W, 1/16W Chip Resistor 0402 (1005 Metric)"
+			(at 49.53 80.01 0)
+			(hide yes)
+			(show_name no)
+			(do_not_autoplace no)
+			(effects
+				(font
+					(size 1.27 1.27)
+				)
+			)
+		)
+		(property "Mfg Part #" "RC0402FR-0710KL"
+			(at 49.53 80.01 0)
+			(hide yes)
+			(show_name no)
+			(do_not_autoplace no)
+			(effects
+				(font
+					(size 1.27 1.27)
+				)
+			)
+		)
+		(property "Manufacturer" "YAGEO"
+			(at 49.53 80.01 0)
+			(hide yes)
+			(show_name no)
+			(do_not_autoplace no)
+			(effects
+				(font
+					(size 1.27 1.27)
+				)
+			)
+		)
+		(property "mpn" "ERJ-2RKF1001X"
+			(at 49.53 80.01 0)
+			(hide yes)
+			(show_name no)
+			(do_not_autoplace no)
+			(effects
+				(font
+					(size 1.27 1.27)
+				)
+			)
+		)
+		(pin "1"
+		)
+		(pin "2"
+		)
+		(instances
+			(project "enchantiS3"
+				(path "/1e57a4ff-0c95-4e2b-9e56-d9bf8e99c9a1/ee30c7d7-fa17-4757-a347-33eaa73dc899"
+					(reference "R19")
+					(unit 1)
+				)
